Commit message: Bugfix & Migration: retargeting model is Wuji Hand 2, not Hand 1
wuji-retargeting pinned to v2026.8.17 for link_naming and chain-resolved PIP/DIP
official Beta 2 URDFs replace the Hand 1 pair, plus the 178 deg root-frame correction
qpos remapped from Pinocchio order to device order before publishing

File: src/wujihand_urdf/wujihand_left.urdf (robot description, URDF)
Before this commit: robot wujihand-left-v1.0.0, 26 links, 25 joints
Links:
- removed link finger1_link1
- removed link finger1_link2
- removed link finger1_link3
- removed link finger1_link4
- removed link finger1_tip_link
- removed link finger2_link1
- removed link finger2_link2
- removed link finger2_link3
- removed link finger2_link4
- removed link finger2_tip_link
- removed link finger3_link1
- removed link finger3_link2
- removed link finger3_link3
- removed link finger3_link4
- removed link finger3_tip_link
- removed link finger4_link1
- removed link finger4_link2
- removed link finger4_link3
- removed link finger4_link4
- removed link finger4_tip_link
- removed link finger5_link1
- removed link finger5_link2
- removed link finger5_link3
- removed link finger5_link4
- removed link finger5_tip_link
- removed link palm_link
- added link l_index_finger_distal, mass 0.005; collision mesh filename=../meshes/left/l_index_finger_distal.STL; visual mesh filename=../meshes/left/l_index_finger_distal.STL
- added link l_index_finger_middle, mass 0.0212; collision mesh filename=../meshes/left/l_index_finger_middle.STL; visual mesh filename=../meshes/left/l_index_finger_middle.STL
- added link l_index_finger_proximal, mass 0.0116; collision mesh filename=../meshes/left/l_index_finger_proximal.STL; visual mesh filename=../meshes/left/l_index_finger_proximal.STL
- added link l_index_finger_proximal_abd, mass 0.0339; collision mesh filename=../meshes/left/l_index_finger_proximal_abd.STL; visual mesh filename=../meshes/left/l_index_finger_proximal_abd.STL
- added link l_index_finger_tip
- added link l_index_finger_tip_sensor_frame, mass 0.003; collision mesh filename=../meshes/left/l_index_finger_tip_sensor_frame.STL; visual mesh filename=../meshes/left/l_index_finger_tip_sensor_frame.STL
- added link l_middle_finger_distal, mass 0.005; collision mesh filename=../meshes/left/l_middle_finger_distal.STL; visual mesh filename=../meshes/left/l_middle_finger_distal.STL
- added link l_middle_finger_middle, mass 0.0212; collision mesh filename=../meshes/left/l_middle_finger_middle.STL; visual mesh filename=../meshes/left/l_middle_finger_middle.STL
- added link l_middle_finger_proximal, mass 0.0116; collision mesh filename=../meshes/left/l_middle_finger_proximal.STL; visual mesh filename=../meshes/left/l_middle_finger_proximal.STL
- added link l_middle_finger_proximal_abd, mass 0.0339; collision mesh filename=../meshes/left/l_middle_finger_proximal_abd.STL; visual mesh filename=../meshes/left/l_middle_finger_proximal_abd.STL
- added link l_middle_finger_tip
- added link l_middle_finger_tip_sensor_frame, mass 0.003; collision mesh filename=../meshes/left/l_middle_finger_tip_sensor_frame.STL; visual mesh filename=../meshes/left/l_middle_finger_tip_sensor_frame.STL
- added link l_pinky_distal, mass 0.005; collision mesh filename=../meshes/left/l_pinky_distal.STL; visual mesh filename=../meshes/left/l_pinky_distal.STL
- added link l_pinky_middle, mass 0.0188; collision mesh filename=../meshes/left/l_pinky_middle.STL; visual mesh filename=../meshes/left/l_pinky_middle.STL
- added link l_pinky_proximal, mass 0.0116; collision mesh filename=../meshes/left/l_pinky_proximal.STL; visual mesh filename=../meshes/left/l_pinky_proximal.STL
- added link l_pinky_proximal_abd, mass 0.0304; collision mesh filename=../meshes/left/l_pinky_proximal_abd.STL; visual mesh filename=../meshes/left/l_pinky_proximal_abd.STL
- added link l_pinky_tip
- added link l_pinky_tip_sensor_frame, mass 0.003; collision mesh filename=../meshes/left/l_pinky_tip_sensor_frame.STL; visual mesh filename=../meshes/left/l_pinky_tip_sensor_frame.STL
- added link l_ring_finger_distal, mass 0.005; collision mesh filename=../meshes/left/l_ring_finger_distal.STL; visual mesh filename=../meshes/left/l_ring_finger_distal.STL
- added link l_ring_finger_middle, mass 0.0212; collision mesh filename=../meshes/left/l_ring_finger_middle.STL; visual mesh filename=../meshes/left/l_ring_finger_middle.STL
- added link l_ring_finger_proximal, mass 0.0116; collision mesh filename=../meshes/left/l_ring_finger_proximal.STL; visual mesh filename=../meshes/left/l_ring_finger_proximal.STL
- added link l_ring_finger_proximal_abd, mass 0.0339; collision mesh filename=../meshes/left/l_ring_finger_proximal_abd.STL; visual mesh filename=../meshes/left/l_ring_finger_proximal_abd.STL
- added link l_ring_finger_tip
- added link l_ring_finger_tip_sensor_frame, mass 0.003; collision mesh filename=../meshes/left/l_ring_finger_tip_sensor_frame.STL; visual mesh filename=../meshes/left/l_ring_finger_tip_sensor_frame.STL
- added link l_thumb_distal, mass 0.0109; collision mesh filename=../meshes/left/l_thumb_distal.STL; visual mesh filename=../meshes/left/l_thumb_distal.STL
- added link l_thumb_middle, mass 0.0358; collision mesh filename=../meshes/left/l_thumb_middle.STL; visual mesh filename=../meshes/left/l_thumb_middle.STL
- added link l_thumb_proximal, mass 0.011; collision mesh filename=../meshes/left/l_thumb_proximal.STL; visual mesh filename=../meshes/left/l_thumb_proximal.STL
- added link l_thumb_proximal_abd, mass 0.0336; collision mesh filename=../meshes/left/l_thumb_proximal_abd.STL; visual mesh filename=../meshes/left/l_thumb_proximal_abd.STL
- added link l_thumb_tip
- added link l_thumb_tip_sensor_frame, mass 0.0063; collision mesh filename=../meshes/left/l_thumb_tip_sensor_frame.STL; visual mesh filename=../meshes/left/l_thumb_tip_sensor_frame.STL
- added link l_wrist, mass 0.2323; collision mesh filename=../meshes/left/l_wrist.STL; visual mesh filename=../meshes/left/l_wrist.STL
Joints:
- removed joint finger1_joint1
- removed joint finger1_joint2
- removed joint finger1_joint3
- removed joint finger1_joint4
- removed joint finger1_tip_fixed
- removed joint finger2_joint1
- removed joint finger2_joint2
- removed joint finger2_joint3
- removed joint finger2_joint4
- removed joint finger2_tip_fixed
- removed joint finger3_joint1
- removed joint finger3_joint2
- removed joint finger3_joint3
- removed joint finger3_joint4
- removed joint finger3_tip_fixed
- removed joint finger4_joint1
- removed joint finger4_joint2
- removed joint finger4_joint3
- removed joint finger4_joint4
- removed joint finger4_tip_fixed
- removed joint finger5_joint1
- removed joint finger5_joint2
- removed joint finger5_joint3
- removed joint finger5_joint4
- removed joint finger5_tip_fixed
- added joint l_index_finger_dip: type revolute, parent l_index_finger_middle, child l_index_finger_distal, origin xyz=0 0 -0.0295 rpy=0 0 0, axis -1 0 0, limit lower=-1.0470 upper=1.5700 effort=0.3000 velocity=13.5
- added joint l_index_finger_mcp_abd: type revolute, parent l_index_finger_proximal, child l_index_finger_proximal_abd, origin xyz=0 0.00120098019222331 -0.014499999983839 rpy=0 0 0, axis 0 1 0, limit lower=-0.6980 upper=0.6980 effort=0.2000 velocity=8.11
- added joint l_index_finger_mcp_flex: type revolute, parent l_wrist, child l_index_finger_proximal, origin xyz=0.0226524150577227 0.00332515884504703 -0.0699780241478046 rpy=0.0397801377022703 -0.136929341252724 -0.100403924639931, axis -1 0 0, limit lower=-1.0470 upper=1.5700 effort=2.0000 velocity=8.203
- added joint l_index_finger_pip: type revolute, parent l_index_finger_proximal_abd, child l_index_finger_middle, origin xyz=0 0 -0.0376 rpy=0 0 0, axis -1 0 0, limit lower=-1.0470 upper=2.0940 effort=0.3000 velocity=12.86
- added joint l_index_finger_tip_fixed: type fixed, parent l_index_finger_distal, child l_index_finger_tip, origin xyz=0 0 -0.02475 rpy=0 0 0
- added joint l_index_finger_tip_sensor_frame_fixed: type fixed, parent l_index_finger_distal, child l_index_finger_tip_sensor_frame, origin xyz=0 0 0 rpy=0 0 0
- added joint l_middle_finger_dip: type revolute, parent l_middle_finger_middle, child l_middle_finger_distal, origin xyz=0 0 -0.0295 rpy=0 0 0, axis -1 0 0, limit lower=-1.0470 upper=1.5700 effort=0.3000 velocity=13.5
- added joint l_middle_finger_mcp_abd: type revolute, parent l_middle_finger_proximal, child l_middle_finger_proximal_abd, origin xyz=0 0.00120098019222334 -0.0144999999838389 rpy=0 0 0, axis 0 1 0, limit lower=-0.6980 upper=0.6980 effort=0.2000 velocity=8.11
- added joint l_middle_finger_mcp_flex: type revolute, parent l_wrist, child l_middle_finger_proximal, origin xyz=0.00094309364603887 0.0083030134913478 -0.0739154421481339 rpy=0.033913594707111 0.011157971722942 0.000715284906568205, axis -1 0 0, limit lower=-1.0470 upper=1.5700 effort=2.0000 velocity=8.203
- added joint l_middle_finger_pip: type revolute, parent l_middle_finger_proximal_abd, child l_middle_finger_middle, origin xyz=0 0 -0.0376 rpy=0 0 0, axis -1 0 0, limit lower=-1.0470 upper=2.0940 effort=0.3000 velocity=12.86
- added joint l_middle_finger_tip_fixed: type fixed, parent l_middle_finger_distal, child l_middle_finger_tip, origin xyz=0 0 -0.02475 rpy=0 0 0
- added joint l_middle_finger_tip_sensor_frame_fixed: type fixed, parent l_middle_finger_distal, child l_middle_finger_tip_sensor_frame, origin xyz=0 0 0 rpy=0 0 0
- added joint l_pinky_dip: type revolute, parent l_pinky_middle, child l_pinky_distal, origin xyz=0 0 -0.0275 rpy=0 0 0, axis -1 0 0, limit lower=-1.0470 upper=1.5700 effort=0.3000 velocity=13.5
- added joint l_pinky_mcp_abd: type revolute, parent l_pinky_proximal, child l_pinky_proximal_abd, origin xyz=0 0.00120098026250511 -0.0145000000235719 rpy=0 0 0, axis 0 1 0, limit lower=-0.6980 upper=0.6980 effort=0.2000 velocity=8.11
- added joint l_pinky_mcp_flex: type revolute, parent l_wrist, child l_pinky_proximal, origin xyz=-0.0373572872886148 0.000733759922594786 -0.0552917010368086 rpy=0.00981701706873381 0.248975826730062 0.13602514715951, axis -1 0 0, limit lower=-1.0470 upper=1.5700 effort=2.0000 velocity=8.203
- added joint l_pinky_pip: type revolute, parent l_pinky_proximal_abd, child l_pinky_middle, origin xyz=-9.99999999990349E-05 0 -0.0336 rpy=0 0 0, axis -1 0 0, limit lower=-1.0470 upper=2.0940 effort=0.3000 velocity=12.86
- added joint l_pinky_tip_fixed: type fixed, parent l_pinky_distal, child l_pinky_tip, origin xyz=0 0 -0.02475 rpy=0 0 0
- added joint l_pinky_tip_sensor_frame_fixed: type fixed, parent l_pinky_distal, child l_pinky_tip_sensor_frame, origin xyz=0 0 0 rpy=0 0 0
- added joint l_ring_finger_dip: type revolute, parent l_ring_finger_middle, child l_ring_finger_distal, origin xyz=0 0 -0.0295 rpy=0 0 0, axis -1 0 0, limit lower=-1.0470 upper=1.5700 effort=0.3000 velocity=13.5
- added joint l_ring_finger_mcp_abd: type revolute, parent l_ring_finger_proximal, child l_ring_finger_proximal_abd, origin xyz=0 0.00120098019222327 -0.014499999983839 rpy=0 0 0, axis 0 1 0, limit lower=-0.6980 upper=0.6980 effort=0.2000 velocity=8.11
- added joint l_ring_finger_mcp_flex: type revolute, parent l_wrist, child l_ring_finger_proximal, origin xyz=-0.019752 0.0055929 -0.065397 rpy=0.016663 0.14175 0.068321, axis -1 0 0, limit lower=-1.0470 upper=1.5700 effort=2.0000 velocity=8.203
- added joint l_ring_finger_pip: type revolute, parent l_ring_finger_proximal_abd, child l_ring_finger_middle, origin xyz=0 0 -0.0376 rpy=0 0 0, axis -1 0 0, limit lower=-1.0470 upper=2.0940 effort=0.3000 velocity=12.86
- added joint l_ring_finger_tip_fixed: type fixed, parent l_ring_finger_distal, child l_ring_finger_tip, origin xyz=0 0 -0.02475 rpy=0 0 0
- added joint l_ring_finger_tip_sensor_frame_fixed: type fixed, parent l_ring_finger_distal, child l_ring_finger_tip_sensor_frame, origin xyz=0 0 0 rpy=0 0 0
- added joint l_thumb_cmc_abd: type revolute, parent l_thumb_proximal, child l_thumb_proximal_abd, origin xyz=0.00025789 0.00063167 -0.014161 rpy=-0.20529 0.70051 -0.025238, axis 0 1 0, limit lower=-1.4840 upper=0.6980 effort=0.6000 velocity=11.1
- added joint l_thumb_cmc_flex: type revolute, parent l_wrist, child l_thumb_proximal, origin xyz=0.017208 -0.008138 -0.01646 rpy=1.6615 -1.0591 -1.9919, axis -1 0 0, limit lower=-1.1870 upper=1.2910 effort=0.6000 velocity=8.587
- added joint l_thumb_ip: type revolute, parent l_thumb_middle, child l_thumb_distal, origin xyz=0 0 -0.0349999999999976 rpy=0 0 0, axis -1 0 0, limit lower=-1.0470 upper=1.5700 effort=0.3000 velocity=13.5
- added joint l_thumb_mcp: type revolute, parent l_thumb_proximal_abd, child l_thumb_middle, origin xyz=-4.31364606099851E-05 2.49048674495827E-05 -0.0334956422241401 rpy=0 0.0872664625997161 -0.523598775598299, axis -1 0 0, limit lower=-1.0470 upper=1.5700 effort=0.3000 velocity=12.86
- added joint l_thumb_tip_fixed: type fixed, parent l_thumb_distal, child l_thumb_tip, origin xyz=0 0 -0.029787 rpy=0 0 0
- added joint l_thumb_tip_sensor_frame_fixed: type fixed, parent l_thumb_distal, child l_thumb_tip_sensor_frame, origin xyz=0 0 0 rpy=0 0 0
