Commit message: Bugfix & Migration: retargeting model is Wuji Hand 2, not Hand 1
wuji-retargeting pinned to v2026.8.17 for link_naming and chain-resolved PIP/DIP
official Beta 2 URDFs replace the Hand 1 pair, plus the 178 deg root-frame correction
qpos remapped from Pinocchio order to device order before publishing

File: src/wujihand_urdf/wujihand_right.urdf (robot description, URDF)
Before this commit: robot wujihand-right-v1.0.0, 26 links, 25 joints
Links:
- removed link finger1_link1
- removed link finger1_link2
- removed link finger1_link3
- removed link finger1_link4
- removed link finger1_tip_link
- removed link finger2_link1
- removed link finger2_link2
- removed link finger2_link3
- removed link finger2_link4
- removed link finger2_tip_link
- removed link finger3_link1
- removed link finger3_link2
- removed link finger3_link3
- removed link finger3_link4
- removed link finger3_tip_link
- removed link finger4_link1
- removed link finger4_link2
- removed link finger4_link3
- removed link finger4_link4
- removed link finger4_tip_link
- removed link finger5_link1
- removed link finger5_link2
- removed link finger5_link3
- removed link finger5_link4
- removed link finger5_tip_link
- removed link palm_link
- added link r_index_finger_distal, mass 0.005; collision mesh filename=../meshes/right/r_index_finger_distal.STL; visual mesh filename=../meshes/right/r_index_finger_distal.STL
- added link r_index_finger_middle, mass 0.0212; collision mesh filename=../meshes/right/r_index_finger_middle.STL; visual mesh filename=../meshes/right/r_index_finger_middle.STL
- added link r_index_finger_proximal, mass 0.0116; collision mesh filename=../meshes/right/r_index_finger_proximal.STL; visual mesh filename=../meshes/right/r_index_finger_proximal.STL
- added link r_index_finger_proximal_abd, mass 0.0339; collision mesh filename=../meshes/right/r_index_finger_proximal_abd.STL; visual mesh filename=../meshes/right/r_index_finger_proximal_abd.STL
- added link r_index_finger_tip
- added link r_index_finger_tip_sensor_frame, mass 0.003; collision mesh filename=../meshes/right/r_index_finger_tip_sensor_frame.STL; visual mesh filename=../meshes/right/r_index_finger_tip_sensor_frame.STL
- added link r_middle_finger_distal, mass 0.005; collision mesh filename=../meshes/right/r_middle_finger_distal.STL; visual mesh filename=../meshes/right/r_middle_finger_distal.STL
- added link r_middle_finger_middle, mass 0.0212; collision mesh filename=../meshes/right/r_middle_finger_middle.STL; visual mesh filename=../meshes/right/r_middle_finger_middle.STL
- added link r_middle_finger_proximal, mass 0.0116; collision mesh filename=../meshes/right/r_middle_finger_proximal.STL; visual mesh filename=../meshes/right/r_middle_finger_proximal.STL
- added link r_middle_finger_proximal_abd, mass 0.0339; collision mesh filename=../meshes/right/r_middle_finger_proximal_abd.STL; visual mesh filename=../meshes/right/r_middle_finger_proximal_abd.STL
- added link r_middle_finger_tip
- added link r_middle_finger_tip_sensor_frame, mass 0.003; collision mesh filename=../meshes/right/r_middle_finger_tip_sensor_frame.STL; visual mesh filename=../meshes/right/r_middle_finger_tip_sensor_frame.STL
- added link r_pinky_distal, mass 0.005; collision mesh filename=../meshes/right/r_pinky_distal.STL; visual mesh filename=../meshes/right/r_pinky_distal.STL
- added link r_pinky_middle, mass 0.0188; collision mesh filename=../meshes/right/r_pinky_middle.STL; visual mesh filename=../meshes/right/r_pinky_middle.STL
- added link r_pinky_proximal, mass 0.0116; collision mesh filename=../meshes/right/r_pinky_proximal.STL; visual mesh filename=../meshes/right/r_pinky_proximal.STL
- added link r_pinky_proximal_abd, mass 0.0304; collision mesh filename=../meshes/right/r_pinky_proximal_abd.STL; visual mesh filename=../meshes/right/r_pinky_proximal_abd.STL
- added link r_pinky_tip
- added link r_pinky_tip_sensor_frame, mass 0.003; collision mesh filename=../meshes/right/r_pinky_tip_sensor_frame.STL; visual mesh filename=../meshes/right/r_pinky_tip_sensor_frame.STL
- added link r_ring_finger_distal, mass 0.005; collision mesh filename=../meshes/right/r_ring_finger_distal.STL; visual mesh filename=../meshes/right/r_ring_finger_distal.STL
- added link r_ring_finger_middle, mass 0.0212; collision mesh filename=../meshes/right/r_ring_finger_middle.STL; visual mesh filename=../meshes/right/r_ring_finger_middle.STL
- added link r_ring_finger_proximal, mass 0.0116; collision mesh filename=../meshes/right/r_ring_finger_proximal.STL; visual mesh filename=../meshes/right/r_ring_finger_proximal.STL
- added link r_ring_finger_proximal_abd, mass 0.0339; collision mesh filename=../meshes/right/r_ring_finger_proximal_abd.STL; visual mesh filename=../meshes/right/r_ring_finger_proximal_abd.STL
- added link r_ring_finger_tip
- added link r_ring_finger_tip_sensor_frame, mass 0.003; collision mesh filename=../meshes/right/r_ring_finger_tip_sensor_frame.STL; visual mesh filename=../meshes/right/r_ring_finger_tip_sensor_frame.STL
- added link r_thumb_distal, mass 0.0109; collision mesh filename=../meshes/right/r_thumb_distal.STL; visual mesh filename=../meshes/right/r_thumb_distal.STL
- added link r_thumb_middle, mass 0.0358; collision mesh filename=../meshes/right/r_thumb_middle.STL; visual mesh filename=../meshes/right/r_thumb_middle.STL
- added link r_thumb_proximal, mass 0.011; collision mesh filename=../meshes/right/r_thumb_proximal.STL; visual mesh filename=../meshes/right/r_thumb_proximal.STL
- added link r_thumb_proximal_abd, mass 0.0336; collision mesh filename=../meshes/right/r_thumb_proximal_abd.STL; visual mesh filename=../meshes/right/r_thumb_proximal_abd.STL
- added link r_thumb_tip
- added link r_thumb_tip_sensor_frame, mass 0.0063; collision mesh filename=../meshes/right/r_thumb_tip_sensor_frame.STL; visual mesh filename=../meshes/right/r_thumb_tip_sensor_frame.STL
- added link r_wrist, mass 0.2323; collision mesh filename=../meshes/right/r_wrist.STL; visual mesh filename=../meshes/right/r_wrist.STL
Joints:
- removed joint finger1_joint1
- removed joint finger1_joint2
- removed joint finger1_joint3
- removed joint finger1_joint4
- removed joint finger1_tip_fixed
- removed joint finger2_joint1
- removed joint finger2_joint2
- removed joint finger2_joint3
- removed joint finger2_joint4
- removed joint finger2_tip_fixed
- removed joint finger3_joint1
- removed joint finger3_joint2
- removed joint finger3_joint3
- removed joint finger3_joint4
- removed joint finger3_tip_fixed
- removed joint finger4_joint1
- removed joint finger4_joint2
- removed joint finger4_joint3
- removed joint finger4_joint4
- removed joint finger4_tip_fixed
- removed joint finger5_joint1
- removed joint finger5_joint2
- removed joint finger5_joint3
- removed joint finger5_joint4
- removed joint finger5_tip_fixed
- added joint r_index_finger_dip: type revolute, parent r_index_finger_middle, child r_index_finger_distal, origin xyz=0 0 -0.0295 rpy=0 0 0, axis 1 0 0, limit lower=-1.0470 upper=1.5700 effort=0.3000 velocity=13.5
- added joint r_index_finger_mcp_abd: type revolute, parent r_index_finger_proximal, child r_index_finger_proximal_abd, origin xyz=0 -0.001201 -0.0145 rpy=0 0 0, axis 0 1 0, limit lower=-0.6980 upper=0.6980 effort=0.2000 velocity=8.11
- added joint r_index_finger_mcp_flex: type revolute, parent r_wrist, child r_index_finger_proximal, origin xyz=0.022661 -0.0033252 -0.069975 rpy=-0.039792 -0.13705 0.10041, axis 1 0 0, limit lower=-1.0470 upper=1.5700 effort=2.0000 velocity=8.203
- added joint r_index_finger_pip: type revolute, parent r_index_finger_proximal_abd, child r_index_finger_middle, origin xyz=0 0 -0.0376 rpy=0 0 0, axis 1 0 0, limit lower=-1.0470 upper=2.0940 effort=0.3000 velocity=12.86
- added joint r_index_finger_tip_fixed: type fixed, parent r_index_finger_distal, child r_index_finger_tip, origin xyz=0 0 -0.02475 rpy=0 0 0
- added joint r_index_finger_tip_sensor_frame_fixed: type fixed, parent r_index_finger_distal, child r_index_finger_tip_sensor_frame, origin xyz=0 0 0 rpy=0 0 0
- added joint r_middle_finger_dip: type revolute, parent r_middle_finger_middle, child r_middle_finger_distal, origin xyz=0 0 -0.0295 rpy=0 0 0, axis 1 0 0, limit lower=-1.0470 upper=1.5700 effort=0.3000 velocity=13.5
- added joint r_middle_finger_mcp_abd: type revolute, parent r_middle_finger_proximal, child r_middle_finger_proximal_abd, origin xyz=0 -0.001201 -0.0145 rpy=0 0 0, axis 0 1 0, limit lower=-0.6980 upper=0.6980 effort=0.2000 velocity=8.11
- added joint r_middle_finger_mcp_flex: type revolute, parent r_wrist, child r_middle_finger_proximal, origin xyz=0.00095202 -0.008303 -0.073915 rpy=-0.03391 0.011037 -0.00071534, axis 1 0 0, limit lower=-1.0470 upper=1.5700 effort=2.0000 velocity=8.203
- added joint r_middle_finger_pip: type revolute, parent r_middle_finger_proximal_abd, child r_middle_finger_middle, origin xyz=0 0 -0.0376 rpy=0 0 0, axis 1 0 0, limit lower=-1.0470 upper=2.0940 effort=0.3000 velocity=12.86
- added joint r_middle_finger_tip_fixed: type fixed, parent r_middle_finger_distal, child r_middle_finger_tip, origin xyz=0 0 -0.02475 rpy=0 0 0
- added joint r_middle_finger_tip_sensor_frame_fixed: type fixed, parent r_middle_finger_distal, child r_middle_finger_tip_sensor_frame, origin xyz=0 0 0 rpy=0 0 0
- added joint r_pinky_dip: type revolute, parent r_pinky_middle, child r_pinky_distal, origin xyz=0 0 -0.0275 rpy=0 0 0, axis 1 0 0, limit lower=-1.0470 upper=1.5700 effort=0.3000 velocity=13.5
- added joint r_pinky_mcp_abd: type revolute, parent r_pinky_proximal, child r_pinky_proximal_abd, origin xyz=0 -0.001201 -0.0145 rpy=0 0 3.6273E-05, axis 0 1 0, limit lower=-0.6980 upper=0.6980 effort=0.2000 velocity=8.11
- added joint r_pinky_mcp_flex: type revolute, parent r_wrist, child r_pinky_proximal, origin xyz=-0.037351 -0.00073376 -0.055296 rpy=-0.029938 0.24886 -0.13602, axis 1 0 0, limit lower=-1.0470 upper=1.5700 effort=2.0000 velocity=8.203
- added joint r_pinky_pip: type revolute, parent r_pinky_proximal_abd, child r_pinky_middle, origin xyz=0.0001 0 -0.0336 rpy=0 0 -3.6273E-05, axis 1 0 0, limit lower=-1.0470 upper=2.0940 effort=0.3000 velocity=12.86
- added joint r_pinky_tip_fixed: type fixed, parent r_pinky_distal, child r_pinky_tip, origin xyz=0 0 -0.02475 rpy=0 0 0
- added joint r_pinky_tip_sensor_frame_fixed: type fixed, parent r_pinky_distal, child r_pinky_tip_sensor_frame, origin xyz=0 0 0 rpy=0 0 0
- added joint r_ring_finger_dip: type revolute, parent r_ring_finger_middle, child r_ring_finger_distal, origin xyz=0 0 -0.0295 rpy=0 0 0, axis 1 0 0, limit lower=-1.0470 upper=1.5700 effort=0.3000 velocity=13.5
- added joint r_ring_finger_mcp_abd: type revolute, parent r_ring_finger_proximal, child r_ring_finger_proximal_abd, origin xyz=0 -0.001201 -0.0145 rpy=0 0 0, axis 0 1 0, limit lower=-0.6980 upper=0.6980 effort=0.2000 velocity=8.11
- added joint r_ring_finger_mcp_flex: type revolute, parent r_wrist, child r_ring_finger_proximal, origin xyz=-0.019744 -0.0055929 -0.0654 rpy=-0.016655 0.14163 -0.06832, axis 1 0 0, limit lower=-1.0470 upper=1.5700 effort=2.0000 velocity=8.203
- added joint r_ring_finger_pip: type revolute, parent r_ring_finger_proximal_abd, child r_ring_finger_middle, origin xyz=0 0 -0.0376 rpy=0 0 0, axis 1 0 0, limit lower=-1.0470 upper=2.0940 effort=0.3000 velocity=12.86
- added joint r_ring_finger_tip_fixed: type fixed, parent r_ring_finger_distal, child r_ring_finger_tip, origin xyz=0 0 -0.02475 rpy=0 0 0
- added joint r_ring_finger_tip_sensor_frame_fixed: type fixed, parent r_ring_finger_distal, child r_ring_finger_tip_sensor_frame, origin xyz=0 0 0 rpy=0 0 0
- added joint r_thumb_cmc_abd: type revolute, parent r_thumb_proximal, child r_thumb_proximal_abd, origin xyz=0.00024788 -0.00053658 -0.014754 rpy=0.20529 0.70051 0.025238, axis 0 1 0, limit lower=-1.4840 upper=0.6980 effort=0.6000 velocity=11.1
- added joint r_thumb_cmc_flex: type revolute, parent r_wrist, child r_thumb_proximal, origin xyz=0.01721 0.008138 -0.016458 rpy=-1.6617 -1.059 1.9921, axis 1 0 0, limit lower=-1.1870 upper=1.2910 effort=0.6000 velocity=8.587
- added joint r_thumb_ip: type revolute, parent r_thumb_middle, child r_thumb_distal, origin xyz=-5E-05 0 -0.035 rpy=0 0 0, axis 1 0 0, limit lower=-1.0470 upper=1.5700 effort=0.3000 velocity=13.5
- added joint r_thumb_mcp: type revolute, parent r_thumb_proximal_abd, child r_thumb_middle, origin xyz=0 0 -0.0325 rpy=0 0.087266 0.56723, axis 1 0 0, limit lower=-1.0470 upper=1.5700 effort=0.3000 velocity=12.86
- added joint r_thumb_tip_fixed: type fixed, parent r_thumb_distal, child r_thumb_tip, origin xyz=0 0 -0.02978 rpy=0 0 0
- added joint r_thumb_tip_sensor_frame_fixed: type fixed, parent r_thumb_distal, child r_thumb_tip_sensor_frame, origin xyz=0 0 0 rpy=0 0 0
