Commit message: feat: mount hands via g1 hand dock link

File: src/g1_wuji2_description/deprecated/no_dock/g1_23_wuji2.urdf (robot description, URDF)
Before this commit: robot g1_23_wuji2, 97 links, 96 joints
Links:
- removed link left_hand_dock
- removed link right_hand_dock
Joints:
- removed joint left_hand_dock_joint
- removed joint right_hand_dock_joint
- joint left_wuji_mount_joint: origin xyz=0.00375 0 0 rpy=0 -1.5707963267948966 0 -> xyz=0.122 0.003 0.0 rpy=0 -1.5707963267948966 0; parent left_hand_dock -> left_wrist_roll_rubber_hand
- joint right_wuji_mount_joint: origin xyz=0.00375 0 0 rpy=0 -1.5707963267948966 0 -> xyz=0.122 -0.003 0.0 rpy=0 -1.5707963267948966 0; parent right_hand_dock -> right_wrist_roll_rubber_hand

File: src/g1_wuji2_description/deprecated/no_dock/g1_29_wuji2.urdf (robot description, URDF)
Before this commit: robot g1_23_wuji2, 97 links, 96 joints
Links:
- removed link left_hand_dock
- removed link left_wrist_roll_rubber_hand
- removed link right_hand_dock
- removed link right_wrist_roll_rubber_hand
- added link left_wrist_pitch_link, mass 0.48404956; collision mesh filename=meshes/g1/left_wrist_pitch_link.STL; visual mesh filename=meshes/g1/left_wrist_pitch_link.STL
- added link left_wrist_roll_link, mass 0.08544498; collision mesh filename=meshes/g1/left_wrist_roll_link.STL; visual mesh filename=meshes/g1/left_wrist_roll_link.STL
- added link left_wrist_yaw_link, mass 0.08457647; collision mesh filename=meshes/g1/left_wrist_yaw_link.STL; visual mesh filename=meshes/g1/left_wrist_yaw_link.STL
- added link right_wrist_pitch_link, mass 0.48404956; collision mesh filename=meshes/g1/right_wrist_pitch_link.STL; visual mesh filename=meshes/g1/right_wrist_pitch_link.STL
- added link right_wrist_roll_link, mass 0.08544498; collision mesh filename=meshes/g1/right_wrist_roll_link.STL; visual mesh filename=meshes/g1/right_wrist_roll_link.STL
- added link right_wrist_yaw_link, mass 0.08457647; collision mesh filename=meshes/g1/right_wrist_yaw_link.STL; visual mesh filename=meshes/g1/right_wrist_yaw_link.STL
- added link waist_roll_link, mass 0.086; visual mesh filename=meshes/g1/waist_roll_link_rev_1_0.STL
- added link waist_yaw_link, mass 0.214; visual mesh filename=meshes/g1/waist_yaw_link_rev_1_0.STL
- link torso_link: geometry collision mesh filename=meshes/g1/torso_link_rev_1_0.STL; visual mesh filename=meshes/g1/torso_link_rev_1_0.STL
Joints:
- removed joint left_hand_dock_joint
- removed joint right_hand_dock_joint
- added joint left_wrist_pitch_joint: type revolute, parent left_wrist_roll_link, child left_wrist_pitch_link, origin xyz=0.038 0 0 rpy=0 0 0, axis 0 1 0, limit lower=-1.614429558 upper=1.614429558 effort=5 velocity=22
- added joint left_wrist_yaw_joint: type revolute, parent left_wrist_pitch_link, child left_wrist_yaw_link, origin xyz=0.046 0 0 rpy=0 0 0, axis 0 0 1, limit lower=-1.614429558 upper=1.614429558 effort=5 velocity=22
- added joint right_wrist_pitch_joint: type revolute, parent right_wrist_roll_link, child right_wrist_pitch_link, origin xyz=0.038 0 0 rpy=0 0 0, axis 0 1 0, limit lower=-1.614429558 upper=1.614429558 effort=5 velocity=22
- added joint right_wrist_yaw_joint: type revolute, parent right_wrist_pitch_link, child right_wrist_yaw_link, origin xyz=0.046 0 0 rpy=0 0 0, axis 0 0 1, limit lower=-1.614429558 upper=1.614429558 effort=5 velocity=22
- added joint waist_pitch_joint: type revolute, parent waist_roll_link, child torso_link, origin xyz=0 0 0 rpy=0 0 0, axis 0 1 0, limit lower=-0.52 upper=0.52 effort=35 velocity=30
- added joint waist_roll_joint: type revolute, parent waist_yaw_link, child waist_roll_link, origin xyz=-0.0039635 0 0.044 rpy=0 0 0, axis 1 0 0, limit lower=-0.52 upper=0.52 effort=35 velocity=30
- joint left_wrist_roll_joint: child left_wrist_roll_rubber_hand -> left_wrist_roll_link
- joint left_wuji_mount_joint: origin xyz=0.00375 0 0 rpy=0 -1.5707963267948966 0 -> xyz=0.0415 0.0 0.0 rpy=0 -1.5707963267948966 0; parent left_hand_dock -> left_wrist_yaw_link
- joint right_wrist_roll_joint: child right_wrist_roll_rubber_hand -> right_wrist_roll_link
- joint right_wuji_mount_joint: origin xyz=0.00375 0 0 rpy=0 -1.5707963267948966 0 -> xyz=0.0415 0.0 0.0 rpy=0 -1.5707963267948966 0; parent right_hand_dock -> right_wrist_yaw_link
- joint waist_yaw_joint: child torso_link -> waist_yaw_link; origin xyz=-0.0039635 0 0.044 rpy=0 0 0 -> xyz=0 0 0 rpy=0 0 0
