Commit message: Fix: drop the removed cross plate from the Hand 2 mount

File: src/g1_wuji2_description/g1_23_wuji2.urdf (robot description, URDF)
Before this commit: robot g1_23_wuji2, 95 links, 94 joints
Links:
- link left_wuji_l_mount: mass 0.069 -> 0.0473079583888804; geometry collision mesh filename=meshes/wuji/left/l_mount_no_cross.STL; visual mesh filename=meshes/wuji/left/l_mount_no_cross.STL
- link right_wuji_r_mount: mass 0.069 -> 0.0473078502572986; geometry collision mesh filename=meshes/wuji/right/r_mount_no_cross.STL; visual mesh filename=meshes/wuji/right/r_mount_no_cross.STL

File: src/g1_wuji2_description/g1_29_wuji2.urdf (robot description, URDF)
Before this commit: robot g1_29_wuji2, 101 links, 100 joints
Links:
- link left_wuji_l_mount: mass 0.069 -> 0.0473079583888804; geometry collision mesh filename=meshes/wuji/left/l_mount_no_cross.STL; visual mesh filename=meshes/wuji/left/l_mount_no_cross.STL
- link right_wuji_r_mount: mass 0.069 -> 0.0473078502572986; geometry collision mesh filename=meshes/wuji/right/r_mount_no_cross.STL; visual mesh filename=meshes/wuji/right/r_mount_no_cross.STL
